File: kicad/batterymeter/batterymeter.kicad_sch (KiCad schematic)
At the start: 145 parts, among them J1 Conn_01x02_Female, J2 Conn_01x04_Male, J3 USB_B_Micro, J4 Conn_01x11_Male, J5 Conn_01x02_Male, J6 Conn_01x03_Male, J9 Conn_01x02_Male, Q1 DMN62D0UDW-13, Q2 DMN62D0UDW-13, SW3 SW_Push, SW4 SW_SLLB5, U1 ATtiny3226-SU, U10 CH340E, U11 TLV9062xD, U12 PCA9536D, U13 74AUP1G02, U14 74AUP1G02, U2 I2C_OLED_128x32, U3 MAX4636EUB+, U4 DG4052EEQ-T1-GE3, U5 DG4052EEQ-T1-GE3, U6 OPA4388ID, U7 MCP1642B-33I/MS, U8 74AHC1G08, U9 MAX4636EUB+

Commit message: better doc
Other:
- note added: "2 1 4 3"
- note added: "Test+ Sense Test+ Test- Sense Test-"
- note added: "XS10:"
- note removed: "Test+ Sense Test+"
- note removed: "Test- Sense Test-"
Changed lines of the file:
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@@
     (effects (font (size 1.27 1.27)) (justify left bottom))
   )
-  (text "Test+\nTest+ Sense" (at 17.145 167.005 0)
+  (text "Test+\nTest+ Sense" (at 20.32 167.005 0)
     (effects (font (size 1.27 1.27)) (justify left bottom))
   )
@@
     (effects (font (size 1.27 1.27)) (justify left bottom))
   )
+  (text "XS10:" (at 13.335 180.975 0)
+    (effects (font (size 1.27 1.27)) (justify left bottom))
+  )
   (text "TODO: get charging status" (at 181.61 -17.78 0)
     (effects (font (size 10 10)) (justify left bottom))
@@
     (effects (font (size 1.27 1.27)) (justify left bottom))
   )
+  (text "2\n1\n4\n3" (at 15.24 189.23 0)
+    (effects (font (size 1.27 1.27)) (justify left bottom))
+  )
   (text "OPTION: \"Intelligent\" battery charger connection\nAllows control over battery charging and auto-ON\nIs destined to replace the circuit to the right of this."
     (at 12.7 203.2 0)
@@
     (effects (font (size 1.27 1.27)) (justify left bottom))
   )
-  (text "Test+ Sense\nTest+" (at 17.145 184.785 0)
+  (text "Test+ Sense\nTest+\nTest- Sense\nTest-" (at 20.955 189.23 0)
     (effects (font (size 1.27 1.27)) (justify left bottom))
   )
@@
     (effects (font (size 1.27 1.27)) (justify left bottom))
   )
-  (text "Test- Sense\nTest-" (at 17.145 189.23 0)
-    (effects (font (size 1.27 1.27)) (justify left bottom))
-  )
